File: rgb_underglow.sch (KiCad schematic (older format))
At the start: 34 parts

Commit message: Update: Work on underglow
Parts:
- removed C? (x8): 100n, Capacitor_SMD:C_0603_1608Metric, symbol Device:C
- removed RGB? (x7): WS2812B, LED_SMD:LED_WS2812B_PLCC4_5.0x5.0mm_P3.2mm, symbol LED:WS2812B
- added C20: 100n, Capacitor_SMD:C_0603_1608Metric, symbol Device:C
- gave numbers to parts that had none: 19
Connections:
- net +5V: now also C20.1
- net GND: now also C20.2
