File: steamvan.sch (KiCad schematic (older format))
At the start: 24 parts, among them J1 Conn_01x05_Male, Q1 FMMT493TA, SW1 SW_Push, U1 STM32F303CBTx, U2 TLV70233_SOT23-5, U3 NUF2221W1T2G, Y1 8MHz

Commit message: Update: Files for KiCad 5.1
Parts:
- U2: symbol Regulator_Linear:TLV70233_SOT23-5 -> steamvan-rescue:TLV70233_SOT23-5-Regulator_Linear
Changed lines of the file:
@@
 EESchema Schematic File Version 4
-LIBS:steamvan-cache
-EELAYER 26 0
+EELAYER 30 0
 EELAYER END
 $Descr A4 11693 8268
@@
 $EndComp
 $Comp
-L Regulator_Linear:TLV70233_SOT23-5 U2
+L steamvan-rescue:TLV70233_SOT23-5-Regulator_Linear U2
 U 1 1 5C200B8E
 P 2630 5600
